File: PCB/Starbie.kicad_pcb (KiCad board)
At the start: 2 copper layers, 152.8 x 126.9 mm, 7 parts, among them J1 Conn_01x04_Pin, J2 Conn_01x08_Pin, SW1 SW_Push, SW2 SW_Push, U1 XIAO-ESP32-C3-SMD, U4 DHT11

Commit message: Add files via upload
Parts:
- moved SW1 3.24 mm to (95.8, 83.0)
Routing:
- net /GPIO2: track 45.8 -> 43.2 mm
Changed lines of the file:
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@@
 			(outputformat 1)
 			(mirror no)
-			(drillshape 1)
+			(drillshape 0)
 			(scaleselection 1)
 			(outputdirectory "")
@@
 	(footprint "Button_Switch_Keyboard:SW_Cherry_MX_1.00u_PCB"
 		(layer "F.Cu")
-		(at 92.96 84.42)
+		(at 95.85 82.96)
 		(descr "Cherry MX keyswitch, 1.00u, PCB mount, http://cherryamericas.com/wp-content/uploads/2014/12/mx_cat.pdf")
 		(tags "Cherry MX keyswitch 1.00u PCB")
@@
 	(gr_arc
 		(start 84.264159 98.446335)
-		(mid 85.815722 100.347165)
+		(mid 85.815703 100.347176)
 		(end 85.718968 102.798946)
 		(stroke
@@
 	)
 	(segment
+		(start 129.562654 85.46)
+		(end 139 85.46)
+		(width 0.2)
+		(layer "F.Cu")
+		(net "/GPIO3")
+	)
+	(segment
+		(start 108.5 109.5)
+		(end 108.5 106.522654)
+		(width 0.2)
+		(layer "F.Cu")
+		(net "/GPIO3")
+	)
+	(segment
+		(start 108.5 106.522654)
+		(end 129.562654 85.46)
+		(width 0.2)
+		(layer "F.Cu")
+		(net "/GPIO3")
+	)
+	(segment
 		(start 124.81 68.695)
 		(end 125.2125 69.0975)
@@
 	)
 	(segment
-		(start 92.96 84.42)
-		(end 94.46 82.92)
+		(start 138.96 82.96)
+		(end 139 82.92)
 		(width 0.2)
 		(layer "F.Cu")
@@
 	)
 	(segment
-		(start 94.46 82.92)
-		(end 138.165 82.92)
+		(start 95.85 82.96)
+		(end 138.96 82.96)
 		(width 0.2)
 		(layer "F.Cu")
 		(net "/GPIO2")
 	)
-	(segment
-		(start 129.562654 85.46)
-		(end 139 85.46)
-		(width 0.2)
-		(layer "F.Cu")
-		(net "/GPIO3")
-	)
-	(segment
-		(start 108.5 109.5)
-		(end 108.5 106.522654)
-		(width 0.2)
-		(layer "F.Cu")
-		(net "/GPIO3")
-	)
-	(segment
-		(start 108.5 106.522654)
-		(end 129.562654 85.46)
-		(width 0.2)
-		(layer "F.Cu")
-		(net "/GPIO3")
-	)
 	(zone
